File: hardware/boards/main-control-board/main-control-board.kicad_pcb (KiCad board)
At the start: 2 copper layers, 80.5 x 50 mm, 40 parts, among them J1 Conn_01x02_Pin_Speaker, J2 Conn_OLED, J3 Conn_extension, J4 Conn_extension_2, J7 Conn_ESP32, J8 Conn_ESP32, U1 PCA9685PW,118, U2 HX PZ2.54-3X5P ZZ, U3 MAX98357AETE+T, U4 TPS259571DSGR

Commit message: add extension port
Parts:
- J4: value Conn_extension_2 -> Conn_02x06_Odd_Even; footprint Connector_PinHeader_2.54mm:PinHeader_1x04_P2.54mm_Vertical -> Connector_PinHeader_2.54mm:PinHeader_2x06_P2.54mm_Vertical
- moved R13 13.5 mm to (126.3, 116.0)
- moved D2 13.4 mm to (128.7, 116.0)
- moved C3 12.1 mm to (118.0, 93.8)
- moved C2 11.9 mm to (151.7, 92.8)
- moved NT1 11.7 mm to (146.2, 89.3)
- moved R12 11.0 mm to (122.0, 94.7)
- moved R5 10.7 mm to (146.4, 113.2)
- moved TP1 10.5 mm to (114.0, 107.1)
- moved TP2 10.4 mm to (114.0, 103.8)
- moved U1 10.0 mm to (138.6, 108.1)
- moved U2 10.0 mm to (138.2, 90.5)
- moved J1 10.0 mm to (116.4, 114.4)
- moved R3 10.0 mm to (139.6, 116.1)
- moved R4 10.0 mm to (142.1, 116.1)
- moved U3 10.0 mm to (121.2, 99.5)
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Connections:
- net Net-(J8-Pin_5) renamed /ESP32/GP10
- J4 pad 2: +3.3V -> /ESP32/GP21
- J4 pad 4: /ESP32/GP6 -> /ESP32/GP20
- J8 pad 2: Net-(J8-Pin_2) -> /ESP32/GP7
- J8 pad 3: Net-(J8-Pin_3) -> /ESP32/GP8
- J8 pad 4: Net-(J8-Pin_4) -> /ESP32/GP9
- J8 pad 8: Net-(J8-Pin_8) -> /ESP32/GP20
- J8 pad 9: Net-(J8-Pin_9) -> /ESP32/GP21
Routing:
- net +3.3V: track 126.8 -> 165.5 mm
- net /ESP32/GP9: track 0.00 -> 24.3 mm
- net /I2S_BCLK: track 72.5 -> 95.7 mm, vias 2 -> 3
- net /ESP32/GP8: track 0.00 -> 20.3 mm
- net /I2S_LRC: track 74.3 -> 93.5 mm, vias 2 -> 3
- net /ESP32/GP7: track 0.00 -> 17.3 mm
- net /ESP32/GP20: track 0.00 -> 16.4 mm
- net /ESP32/GP21: track 0.00 -> 14.7 mm
- net /I2C_SCL: track 78.2 -> 89.9 mm
- net GND: track 21.0 -> 9.89 mm, vias 38 -> 41
- net /ESP32/GP5: track 52.8 -> 63.7 mm
- net /I2C_SDA: track 82.6 -> 93.5 mm
- net /PCA/SERVO_5V: track 48.6 -> 59.3 mm
- net /I2S_DIN: track 74.6 -> 83.9 mm
- net /Audio/AUDIO_5V: track 39.9 -> 38.5 mm
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- added copper zone on F.Cu, net /Audio/AUDIO_5V
Other:
- board size 80.5 x 50 mm -> 90.5 x 50 mm
- board text added: "BCLK"
- board text added: "GP20"
- board text added: "GP21"
- board text added: "I2S"
- board text added: "LRC"
- board text added: "TINY SOFTWARE ENGINEER Main Control Board HW REV #3 | 2026-10-06 github.com/jamro/tiny-engineer"
- board text removed: "TINY SOFTWARE ENGINEER Main Control Board HW REV #2 | 2026-09-24 github.com/jamro/tiny-engineer"

Commit message: update BOM
Routing:
- net GND: vias 41 -> 44
